Commit message: updated packages

File: my_robot_description/urdf/robbie.urdf (robot description, URDF)
Before this commit: robot robbie, 12 links, 11 joints
Links:
- link base_link: geometry collision box size=0.07 0.20 0.405; collision box size=0.10 0.05 0.01
Joints:
- joint shoulder_roll: origin xyz=0 0.09 0.22 rpy=0 0 0 -> xyz=0 0.09 0.233 rpy=0 0 0

File: my_robot_description/urdf/robbie.urdf.xacro (robot description, xacro)
@@ -1,8 +1,9 @@
 <?xml version="1.0"?>
 <robot xmlns:xacro="http://www.ros.org/wiki/xacro" name="robbie">
+  <xacro:arg name="initial_positions_file" default="initial_positions.yaml"/>
+  <xacro:arg name="use_real_hardware" default="false"/>
   <xacro:arg name="controller_file" default=""/>
-  <xacro:arg name="initial_positions_file" default=""/>
   <xacro:include filename="$(find my_robot_description)/urdf/robbie.urdf"/>
+  <xacro:include filename="$(find my_robot_description)/urdf/ros2_control.xacro"/>
   <xacro:include filename="$(find my_robot_description)/urdf/gazebo.xacro"/>
-  <xacro:include filename="$(find my_robot_description)/urdf/ros2_control.xacro"/>
 </robot>

File: my_robot_description/urdf/ros2_control.xacro (robot description, xacro)
@@ -1,31 +1,40 @@
 <?xml version="1.0"?>
 <robot xmlns:xacro="http://www.ros.org/wiki/xacro">
-  <ros2_control name="GazeboSystem" type="system">
+  <ros2_control name="ArmHardware" type="system">
     <hardware>
-        <plugin>gz_ros2_control/GazeboSimSystem</plugin>
+      <plugin>my_robot_controller/ArmHardwareInterface</plugin>
+      <param name="serial_port">/dev/ttyACM0</param>
+      <param name="baud_rate">9600</param>
+      <param name="use_serial">true</param>
     </hardware>
     <!-- Arm joints -->
     <joint name="shoulder_roll">
       <command_interface name="position"/>
+        <param name="initial_value">0.0</param>
       <state_interface name="position"/>
     </joint>
     <joint name="shoulder_pitch">
       <command_interface name="position"/>
+        <param name="initial_value">0.5</param>
       <state_interface name="position"/>
     </joint>
     <joint name="elbow_roll">
       <command_interface name="position"/>
+        <param name="initial_value">0.0</param>
       <state_interface name="position"/>
     </joint>
     <joint name="elbow_pitch">
       <command_interface name="position"/>
+        <param name="initial_value">0.5</param>
       <state_interface name="position"/>
     </joint>
     <joint name="wrist_roll">
       <command_interface name="position"/>
+        <param name="initial_value">0.0</param>
       <state_interface name="position"/>
     </joint>
     <joint name="wrist_pitch">
       <command_interface name="position"/>
+        <param name="initial_value">0.0</param>
       <state_interface name="position"/>
     </joint>

File: my_robot_moveit_config/config/robbie.urdf.xacro (robot description, xacro)
@@ -2,8 +2,8 @@
 <robot xmlns:xacro="http://www.ros.org/wiki/xacro" name="robbie">
   <xacro:arg name="initial_positions_file" default="initial_positions.yaml"/>
-  <xacro:arg name="use_gazebo" default="true"/>
-  <xacro:arg name="ros2_controllers_file" default=""/>
+  <xacro:arg name="use_real_hardware" default="false"/>
+  <xacro:arg name="controller_file" default=""/>
   <xacro:include filename="$(find my_robot_description)/urdf/robbie.urdf"/>
-  <xacro:include filename="$(find my_robot_description)/urdf/ros2_control.xacro"/>  <!-- ✅ ADD BACK -->
+  <xacro:include filename="$(find my_robot_description)/urdf/ros2_control.xacro"/>
   <xacro:include filename="$(find my_robot_description)/urdf/gazebo.xacro"/>
 </robot>
